File: eagle/ADS Boards/Main Board.brd (EAGLE design)
At the start: 61.7 x 61.7 mm, 14 parts

Commit message: Finalized Boards, Gerbers, and DXF files.
Parts:
- removed EXTENSION: (no value), con-lstb:MA10-2
- removed U$3: SLIDE_SWITCH, ME433:SLIDE_SWITCH
- added C1: 0.33uF, resistor:C0805
- added C2: 0.1uF, resistor:C0805
- added J1: 62674-121121ALF, NUSTARS ADS Library:CON12_1X12_DUT_58XF
- added R1, R2, R3: 330, resistor:R0805
- added U$4: SLIDE_SWITCH2, ME433:SLIDE_SWITCH2
- moved LED3 4.02 mm to (11.4, 27.9)
- moved LED2 3.59 mm to (14.0, 34.3)
- moved LED1 2.62 mm to (19.7, 39.4)
Connections:
- new net N$1: LED1.K, R1.2
- new net N$3: LED2.K, R2.2
- new net N$4: LED3.K, R3.2
- net 3.3V: now also J1.1; no longer EXTENSION.20
- net 5V: now also C2.1
- net ADR: now also J1.11; no longer EXTENSION.10
- net B1: now also J1.4; no longer EXTENSION.19
- net B2: now also J1.5; no longer EXTENSION.17
- net B3: now also J1.6; no longer EXTENSION.15
- net B4: now also J1.7; no longer EXTENSION.13
- net B5: now also J1.8; no longer EXTENSION.11
- net B6: now also J1.9; no longer EXTENSION.9
- net GND: now also C1.2, C2.2, J1.12, R1.1, R2.1, R3.1, U$4.OUT1; no longer EXTENSION.1, LED1.K, LED2.K, LED3.K, U$3.OUT1
- net RST: now also J1.10; no longer EXTENSION.12
- net SCL: now also J1.3; no longer EXTENSION.16
- net SDA: now also J1.2; no longer EXTENSION.18
- net V_BATT: now also U$4.OUT2; no longer U$3.OUT2
- net V_IN: now also C1.1, U$4.IN; no longer U$3.IN
Routing:
- net GND: track 2.72 -> 21.7 mm, vias 2 -> 10
- net ADR: track 19.6 -> 38.3 mm, vias 2 -> 1
- net RST: track 19.9 -> 29.9 mm
- net ERROR_LED: track 14.4 -> 19.7 mm
- net N$3: track 0.00 -> 4.47 mm
- net N$4: track 0.00 -> 4.47 mm
- net B5: track 34.2 -> 38.1 mm, vias 2 -> 0
- net N$1: track 0.00 -> 3.94 mm
- net B3: track 36.0 -> 39.8 mm
- net STATUS_LED: track 11.0 -> 14.6 mm
- net SCL: track 14.0 -> 17.4 mm, vias 2 -> 1
- net B6: track 31.9 -> 34.9 mm
- net B2: track 36.5 -> 39.0 mm, vias 1 -> 0
- net B4: track 34.2 -> 36.6 mm
- net SDA: track 16.2 -> 18.5 mm
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- added copper zone on layer 1, net V_BATT
- added copper zone on layer 16, net V_BATT
Other:
- board text added: "5V"
- board text added: "7.4V"
- board text added: "ACTIVE DRAG SYSTEM"
- board text added: "BAT"
- board text added: "GND"
- board text added: "Hardware Rev. 1.0"
- board text added: "MAIN BOARD"
- board text added: "MOTOR"
- board text added: "NUSTARS"
