File: eagle/ADS Boards/Main Board.sch (EAGLE design)
At the start: 19 parts, among them J1 62674-121121ALF

Commit message: fixed rocket boards
Parts:
- removed C1: 0.33uF, resistor:C-USC0805
- removed C2: 0.1uF, resistor:C-USC0805
- removed U$2: VREG, NUSTARS ADS Library:VREG
- added C3: 0.33uF, resistor:C-USC0805
- added C4: 0.1uF, resistor:C-USC0805
- added IC1: 7808T, adafruit:7808T
- added J2: (no value), SparkFun-Connectors:CONN_08"
- added LED4: (no value), led:LEDSML0805
- added R4: 330, resistor:R-US_R0805
- LED1, LED2, LED3: device led:LED3MM -> led:LEDSML0805
Connections:
- removed net N$3: LED2.C, R2.2
- removed net POWER_LED: LED1.A, U$1.8
- new net MISC_LED: R4.2, U$1.11
- new net N$5: LED3.A, R3.1
- new net N$6: LED4.A, R4.1
- net 3.3V: now also J2.1, R1.2
- net 5V: now also C4.1, IC1.VO; no longer C2.1, U$2.OUT
- net B3: now also J2.4; no longer J1.66
- net B4: now also J2.5; no longer J1.77
- net B5: now also J2.6; no longer J1.88
- net B6: now also J2.7; no longer J1.99
- net ERROR_LED: now also R3.2; no longer LED3.A
- net GND: now also BATTERY1.2, C3.2, C4.2, IC1.GND, J2.8, LED1.C, LED2.C, LED3.C, LED4.C; no longer BATTERY2.1, C1.2, C2.2, R1.1, R2.1, R3.1, U$2.GND
- net N$1: now also LED1.A, R1.1; no longer LED1.C, R1.2
- net N$4: now also LED2.A, R2.1; no longer LED3.C, R3.2
- net SCL: now also J2.3
- net SDA: now also J2.2
- net STATUS_LED: now also R2.2; no longer LED2.A
- net V_BATT: now also BATTERY2.1; no longer BATTERY1.2, MOTOR.2
- net V_IN: now also C3.1, IC1.VI, MOTOR.2; no longer C1.1, U$2.IN
Other:
- moved on the sheet: BATTERY1, BATTERY2, LED1, LED2, LED3, R1, R2, R3
